File: circuit-diagrams/Layer1_v1.0.brd (EAGLE design)
At the start: 40.6 x 40.6 mm, 41 parts, among them U1 MCP73831, X1 USBSMD

Commit message: Added Layer CircuitCAM, Eagle, BoardMaster files
Parts:
- moved X1 29.0 mm to (18.4, 6.35), turned to 90 degrees
- moved STAT 27.6 mm to (12.7, 1.27), turned to 270 degrees
- moved R16 17.7 mm to (23.5, 12.7), turned to 90 degrees
- moved BATTERY 14.5 mm to (17.1, 22.2)
- moved U1 11.0 mm to (14.0, 12.7), turned to 90 degrees
- moved POWER 8.28 mm to (1.91, 20.3)
- moved C1 6.87 mm to (21.0, 15.9)
- moved R14 5.68 mm to (17.8, 12.1)
- moved C2 4.49 mm to (12.1, 15.9)
Routing:
- net GND: track 82.8 -> 138.9 mm
- net VOUT: track 0.00 -> 46.5 mm
- net N$14: track 0.00 -> 22.5 mm
- net VIN: track 0.00 -> 15.9 mm
- net VCC: track 0.00 -> 13.5 mm
- net STAT: track 0.00 -> 10.7 mm
- net PROG: track 8.93 -> 3.67 mm
- net N$8: track 14.2 -> 15.1 mm

Commit message: Fixed mapping of pins in layer 2 in v1.1
Parts:
- R13: value (none) -> 330
Changed lines of the file:
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@@
 <?xml version="1.0" encoding="utf-8"?>
 <!DOCTYPE eagle SYSTEM "eagle.dtd">
-<eagle version="6.4">
+<eagle version="6.2">
 <drawing>
 <settings>
@@
 <layers>
 <layer number="1" name="Top" color="4" fill="1" visible="yes" active="yes"/>
-<layer number="16" name="Bottom" color="1" fill="1" visible="yes" active="yes"/>
+<layer number="16" name="Bottom" color="1" fill="1" visible="no" active="yes"/>
 <layer number="17" name="Pads" color="2" fill="1" visible="yes" active="yes"/>
 <layer number="18" name="Vias" color="2" fill="1" visible="yes" active="yes"/>
 <layer number="19" name="Unrouted" color="6" fill="1" visible="yes" active="yes"/>
 <layer number="20" name="Dimension" color="15" fill="1" visible="yes" active="yes"/>
-<layer number="21" name="tPlace" color="7" fill="1" visible="no" active="yes"/>
+<layer number="21" name="tPlace" color="7" fill="1" visible="yes" active="yes"/>
 <layer number="22" name="bPlace" color="7" fill="1" visible="yes" active="yes"/>
-<layer number="23" name="tOrigins" color="15" fill="1" visible="no" active="yes"/>
+<layer number="23" name="tOrigins" color="15" fill="1" visible="yes" active="yes"/>
 <layer number="24" name="bOrigins" color="15" fill="1" visible="yes" active="yes"/>
-<layer number="25" name="tNames" color="7" fill="1" visible="no" active="yes"/>
+<layer number="25" name="tNames" color="7" fill="1" visible="yes" active="yes"/>
 <layer number="26" name="bNames" color="7" fill="1" visible="yes" active="yes"/>
-<layer number="27" name="tValues" color="7" fill="1" visible="no" active="yes"/>
+<layer number="27" name="tValues" color="7" fill="1" visible="yes" active="yes"/>
 <layer number="28" name="bValues" color="7" fill="1" visible="yes" active="yes"/>
 <layer number="29" name="tStop" color="7" fill="3" visible="no" active="yes"/>
@@
 </class>
 </classes>
-<designrules name="default">
+<designrules>
 <description language="de">&lt;b&gt;EAGLE Design Rules&lt;/b&gt;
 &lt;p&gt;
@@
 <attribute name="NAME" x="3.7338" y="6.2738" size="1.27" layer="26" ratio="10" rot="MR90"/>
 </element>
-<element name="R13" library="SparkFun-Passives" package="0603-RES" value="" x="31.115" y="33.02" rot="MR270"/>
+<element name="R13" library="SparkFun-Passives" package="0603-RES" value="330" x="31.115" y="33.02" rot="MR270"/>
 <element name="LED13" library="adafruit" package="CHIPLED_0603" value="" x="32.385" y="37.465" smashed="yes" rot="MR90">
 <attribute name="VALUE" x="31.115" y="40.005" size="1.27" layer="28" rot="MR180"/>
@@
 </signal>
 </signals>
-<errors>
-</errors>
 </board>
 </drawing>
